File: banana to usb-A/Banana to USB Adapter.kicad_pcb (KiCad board)
At the start: 2 copper layers, 34.3 x 26.6 mm, 29 parts, among them J1 USB_A, J2 Positive, J3 Negative, J4 Data

Commit message: No design changes to PCB. Removed extra LED reference in schematic, changed TVS diode to D2, and uploaded PCB.
Parts:
- removed ? (x7): , 
- removed REF** (x13): 25mil_Hole, My Libraries:25mil_Hole
