File: banana to barrel jack/Banana to Barrel Jack Adapter.kicad_pcb (KiCad board)
At the start: 2 copper layers, 34.3 x 26.6 mm, 12 parts, among them J1 Barrel_Jack_Switch, J2 Positive, J3 Negative

Commit message: fixed missing drill holes
Parts:
- added ?: , , F.Cu at (136.9, 96.1)
- added ?: , , F.Cu at (136.9, 102.7)
- added ?: , , F.Cu at (136.9, 97.2)
- added ?: , , F.Cu at (136.9, 99.3)
- added ?: , , F.Cu at (136.9, 101.6)
- added ?: , , F.Cu at (136.9, 98.3)
- added ?: , , F.Cu at (136.9, 100.5)
- added REF**: 25mil_Hole, My Libraries:25mil_Hole, F.Cu at (133.0, 99.5)
- added REF**: 25mil_Hole, My Libraries:25mil_Hole, F.Cu at (126.1, 99.5)
- added REF**: 25mil_Hole, My Libraries:25mil_Hole, F.Cu at (133.0, 97.5)
- added REF**: 25mil_Hole, My Libraries:25mil_Hole, F.Cu at (133.0, 101.9)
- added REF**: 25mil_Hole, My Libraries:25mil_Hole, F.Cu at (133.0, 98.6)
- added REF**: 25mil_Hole, My Libraries:25mil_Hole, F.Cu at (133.0, 103.1)
- added REF**: 25mil_Hole, My Libraries:25mil_Hole, F.Cu at (133.0, 96.4)
- added REF**: 25mil_Hole, My Libraries:25mil_Hole, F.Cu at (128.4, 99.5)
- added REF**: 25mil_Hole, My Libraries:25mil_Hole, F.Cu at (127.3, 99.5)
- added REF**: 25mil_Hole, My Libraries:25mil_Hole, F.Cu at (129.6, 99.5)
- added REF**: 25mil_Hole, My Libraries:25mil_Hole, F.Cu at (130.8, 99.5)
- added REF**: 25mil_Hole, My Libraries:25mil_Hole, F.Cu at (133.0, 100.8)
- added REF**: 25mil_Hole, My Libraries:25mil_Hole, F.Cu at (131.9, 99.5)
