File: banana to usb-c/Banana to USB-C Adapter.kicad_sch (KiCad schematic)
At the start: 12 parts, among them J1 USB4125-GF-A-0190, J2 Positive, J3 Negative

Commit message: usb-c ready for fab
Other:
- title: Banana-to-usb adapter -> Banana to USB-C Adapter (Power Only)
Changed lines of the file:
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@@
 	(paper "A4")
 	(title_block
-		(title "Banana-to-usb adapter")
+		(title "Banana to USB-C Adapter (Power Only)")
 		(date "2024-04-06")
 		(rev "2")
